Commit message: change to twist

File: src/vehicle_simulator/urdf/lidar.urdf.xacro (robot description, xacro)
@@ -1,7 +1,11 @@
 <robot xmlns:xacro="http://www.ros.org/wiki/xacro" name="example">
   <link name="lidar" />
-  <xacro:include filename="$(find velodyne_description)/urdf/VLP-16.urdf.xacro"/>
-  <xacro:VLP-16 parent="lidar" name="velodyne" topic="/velodyne_points" hz="5" samples="350" min_range="0.1" organize_cloud="true">
-    <origin xyz="0 0 0" rpy="0 0 0" />
-  </xacro:VLP-16>
+<!--  <xacro:include filename="$(find velodyne_description)/urdf/VLP-16.urdf.xacro"/>-->
+<!--  <xacro:VLP-16 parent="lidar" name="velodyne" topic="/velodyne_points" hz="5" samples="350" min_range="0.1" organize_cloud="true">-->
+<!--    <origin xyz="0 0 0" rpy="0 0 0" />-->
+<!--  </xacro:VLP-16>-->
+    <xacro:include filename="$(find livox_laser_simulation)/urdf/Livox-MID360.urdf.xacro"/>
+    <xacro:Livox-MID360 parent="lidar" name="sensor" topic="/velodyne_points">
+      <origin xyz="0 0 0.07212" rpy="0 0 0" />
+    </xacro:Livox-MID360>
 </robot>
